Commit message: Add official XLeRobot adapter and gripper support

File: src/so101_gazebo/urdf/so101_gazebo.urdf.xacro (robot description, xacro)
@@ -309,5 +309,5 @@
       <origin xyz="0 0 0" rpy="0 0 0"/>
       <mass value="1e-9"/>
-      <inertia ixx="0" ixy="0" ixz="0" iyy="0" iyz="0" izz="0"/>
+      <inertia ixx="1e-9" ixy="0" ixz="0" iyy="1e-9" iyz="0" izz="1e-9"/>
     </inertial>
   </link>

File: src/xlerobot_gazebo/urdf/xlerobot.urdf.xacro (robot description, xacro)
@@ -293,6 +293,6 @@
       lower="-2.1"
       upper="2.1"
-      effort="0"
-      velocity="0" />
+      effort="8.85"
+      velocity="3.14" />
   </joint>
   <link name="Upper_Arm">
@@ -365,6 +365,6 @@
       lower="-0.1"
       upper="3.45"
-      effort="0"
-      velocity="0" />
+      effort="8.85"
+      velocity="3.14" />
   </joint>
   <link name="Lower_Arm">
@@ -426,5 +426,5 @@
     <child link="Lower_Arm" />
     <axis xyz="1 0 0" />
-    <limit lower="-0.2" upper="3.14159" effort="0" velocity="0" />
+    <limit lower="-0.2" upper="3.14159" effort="8.85" velocity="3.14" />
   </joint>
   <link name="Wrist_Pitch_Roll">
@@ -488,6 +488,6 @@
       lower="-1.8"
       upper="1.8"
-      effort="0"
-      velocity="0" />
+      effort="8.85"
+      velocity="3.14" />
   </joint>
   <link name="Fixed_Jaw">
@@ -526,20 +526,11 @@
       </material>
     </visual>
-    <collision>
-      <origin
-        xyz="0 0 0"
-        rpy="0 0 0" />
-      <geometry>
-        <mesh
-          filename="package://xlerobot_gazebo/meshes/Fixed_Jaw_part1.ply" />
-      </geometry>
-    </collision>
-    <collision>
-      <origin
-        xyz="0 0 0"
-        rpy="0 0 0" />
-      <geometry>
-        <mesh
-          filename="package://xlerobot_gazebo/meshes/Fixed_Jaw_part2.ply" />
+    <!-- Simplified collision keeps the gripper movable in Gazebo. -->
+    <collision>
+      <origin
+        xyz="0.008 -0.044 0"
+        rpy="0 0 0" />
+      <geometry>
+        <box size="0.026 0.088 0.028" />
       </geometry>
     </collision>
@@ -550,5 +541,5 @@
     <child link="Fixed_Jaw" />
     <axis xyz="0 -1 0" />
-    <limit lower="-3.14159" upper="3.14159" effort="0" velocity="0" />
+    <limit lower="-3.14159" upper="3.14159" effort="8.85" velocity="3.14" />
   </joint>
   <link name="Moving_Jaw">
@@ -580,27 +571,8 @@
     <collision>
       <origin
-        xyz="0 0 0"
-        rpy="0 0 0" />
-      <geometry>
-        <mesh
-          filename="package://xlerobot_gazebo/meshes/Moving_Jaw_part1.ply" />
-      </geometry>
-    </collision>
-    <collision>
-      <origin
-        xyz="0 0 0"
-        rpy="0 0 0" />
-      <geometry>
-        <mesh
-          filename="package://xlerobot_gazebo/meshes/Moving_Jaw_part2.ply" />
-      </geometry>
-    </collision>
-    <collision>
-      <origin
-        xyz="0 0 0"
-        rpy="0 0 0" />
-      <geometry>
-        <mesh
-          filename="package://xlerobot_gazebo/meshes/Moving_Jaw_part3.ply" />
+        xyz="-0.003 -0.048 0"
+        rpy="0 0 0" />
+      <geometry>
+        <box size="0.018 0.072 0.02" />
       </geometry>
     </collision>
@@ -611,5 +583,6 @@
     <child link="Moving_Jaw" />
     <axis xyz="0 0 1" />
-    <limit lower="0" upper="1.7" effort="0" velocity="0" />
+    <dynamics damping="0.2" friction="0.0" />
+    <limit lower="-3.14159" upper="3.14159" effort="8.85" velocity="3.14" />
   </joint>
   <!-- fake joints for useful data -->
@@ -810,6 +783,6 @@
       lower="-2.1"
       upper="2.1"
-      effort="0"
-      velocity="0" />
+      effort="8.85"
+      velocity="3.14" />
   </joint>
   <link name="Upper_Arm_2">
@@ -880,6 +853,6 @@
       lower="-0.1"
       upper="3.45"
-      effort="0"
-      velocity="0" />
+      effort="8.85"
+      velocity="3.14" />
   </joint>
   <link name="Lower_Arm_2">
@@ -941,5 +914,5 @@
     <child link="Lower_Arm_2" />
     <axis xyz="1 0 0" />
-    <limit lower="-0.2" upper="3.14159" effort="0" velocity="0" />
+    <limit lower="-0.2" upper="3.14159" effort="8.85" velocity="3.14" />
   </joint>
   <link name="Wrist_Pitch_Roll_2">
@@ -1001,6 +974,6 @@
       lower="-1.8"
       upper="1.8"
-      effort="0"
-      velocity="0" />
+      effort="8.85"
+      velocity="3.14" />
   </joint>
   <link name="Fixed_Jaw_2">
@@ -1039,20 +1012,11 @@
       </material>
     </visual>
-    <collision>
-      <origin
-        xyz="0 0 0"
-        rpy="0 0 0" />
-      <geometry>
-        <mesh
-          filename="package://xlerobot_gazebo/meshes/Fixed_Jaw_part1.ply" />
-      </geometry>
-    </collision>
-    <collision>
-      <origin
-        xyz="0 0 0"
-        rpy="0 0 0" />
-      <geometry>
-        <mesh
-          filename="package://xlerobot_gazebo/meshes/Fixed_Jaw_part2.ply" />
+    <!-- Simplified collision keeps the gripper movable in Gazebo. -->
+    <collision>
+      <origin
+        xyz="0.008 -0.044 0"
+        rpy="0 0 0" />
+      <geometry>
+        <box size="0.026 0.088 0.028" />
       </geometry>
     </collision>
@@ -1063,5 +1027,5 @@
     <child link="Fixed_Jaw_2" />
     <axis xyz="0 -1 0" />
-    <limit lower="-3.14159" upper="3.14159" effort="0" velocity="0" />
+    <limit lower="-3.14159" upper="3.14159" effort="8.85" velocity="3.14" />
   </joint>
   <link name="Moving_Jaw_2">
@@ -1090,27 +1054,8 @@
     <collision>
       <origin
-        xyz="0 0 0"
-        rpy="0 0 0" />
-      <geometry>
-        <mesh
-          filename="package://xlerobot_gazebo/meshes/Moving_Jaw_part1.ply" />
-      </geometry>
-    </collision>
-    <collision>
-      <origin
-        xyz="0 0 0"
-        rpy="0 0 0" />
-      <geometry>
-        <mesh
-          filename="package://xlerobot_gazebo/meshes/Moving_Jaw_part2.ply" />
-      </geometry>
-    </collision>
-    <collision>
-      <origin
-        xyz="0 0 0"
-        rpy="0 0 0" />
-      <geometry>
-        <mesh
-          filename="package://xlerobot_gazebo/meshes/Moving_Jaw_part3.ply" />
+        xyz="-0.003 -0.048 0"
+        rpy="0 0 0" />
+      <geometry>
+        <box size="0.018 0.072 0.02" />
       </geometry>
     </collision>
@@ -1121,5 +1066,6 @@
     <child link="Moving_Jaw_2" />
     <axis xyz="0 0 1" />
-    <limit lower="0" upper="1.7" effort="0" velocity="0" />
+    <dynamics damping="0.2" friction="0.0" />
+    <limit lower="-3.14159" upper="3.14159" effort="8.85" velocity="3.14" />
   </joint>
   <!-- fake joints for useful data -->

File: src/xlerobot_gazebo/urdf/xlerobot_planar.urdf.xacro (robot description, xacro)
@@ -280,6 +280,6 @@
       lower="-2.1"
       upper="2.1"
-      effort="0"
-      velocity="0" />
+      effort="8.85"
+      velocity="3.14" />
   </joint>
   <link name="Upper_Arm">
@@ -352,6 +352,6 @@
       lower="-0.1"
       upper="3.45"
-      effort="0"
-      velocity="0" />
+      effort="8.85"
+      velocity="3.14" />
   </joint>
   <link name="Lower_Arm">
@@ -413,5 +413,5 @@
     <child link="Lower_Arm" />
     <axis xyz="1 0 0" />
-    <limit lower="-0.2" upper="3.14159" effort="0" velocity="0" />
+    <limit lower="-0.2" upper="3.14159" effort="8.85" velocity="3.14" />
   </joint>
   <link name="Wrist_Pitch_Roll">
@@ -475,6 +475,6 @@
       lower="-1.8"
       upper="1.8"
-      effort="0"
-      velocity="0" />
+      effort="8.85"
+      velocity="3.14" />
   </joint>
   <link name="Fixed_Jaw">
@@ -513,20 +513,11 @@
       </material>
     </visual>
-    <collision>
-      <origin
-        xyz="0 0 0"
-        rpy="0 0 0" />
-      <geometry>
-        <mesh
-          filename="package://xlerobot_gazebo/meshes/Fixed_Jaw_part1.ply" />
-      </geometry>
-    </collision>
-    <collision>
-      <origin
-        xyz="0 0 0"
-        rpy="0 0 0" />
-      <geometry>
-        <mesh
-          filename="package://xlerobot_gazebo/meshes/Fixed_Jaw_part2.ply" />
+    <!-- Simplified collision keeps the gripper movable in Gazebo. -->
+    <collision>
+      <origin
+        xyz="0.008 -0.044 0"
+        rpy="0 0 0" />
+      <geometry>
+        <box size="0.026 0.088 0.028" />
       </geometry>
     </collision>
@@ -537,5 +528,5 @@
     <child link="Fixed_Jaw" />
     <axis xyz="0 -1 0" />
-    <limit lower="-3.14159" upper="3.14159" effort="0" velocity="0" />
+    <limit lower="-3.14159" upper="3.14159" effort="8.85" velocity="3.14" />
   </joint>
   <link name="Moving_Jaw">
@@ -567,27 +558,8 @@
     <collision>
       <origin
-        xyz="0 0 0"
-        rpy="0 0 0" />
-      <geometry>
-        <mesh
-          filename="package://xlerobot_gazebo/meshes/Moving_Jaw_part1.ply" />
-      </geometry>
-    </collision>
-    <collision>
-      <origin
-        xyz="0 0 0"
-        rpy="0 0 0" />
-      <geometry>
-        <mesh
-          filename="package://xlerobot_gazebo/meshes/Moving_Jaw_part2.ply" />
-      </geometry>
-    </collision>
-    <collision>
-      <origin
-        xyz="0 0 0"
-        rpy="0 0 0" />
-      <geometry>
-        <mesh
-          filename="package://xlerobot_gazebo/meshes/Moving_Jaw_part3.ply" />
+        xyz="-0.003 -0.048 0"
+        rpy="0 0 0" />
+      <geometry>
+        <box size="0.018 0.072 0.02" />
       </geometry>
     </collision>
@@ -598,5 +570,6 @@
     <child link="Moving_Jaw" />
     <axis xyz="0 0 1" />
-    <limit lower="0" upper="1.7" effort="0" velocity="0" />
+    <dynamics damping="0.2" friction="0.0" />
+    <limit lower="-3.14159" upper="3.14159" effort="8.85" velocity="3.14" />
   </joint>
   <!-- fake joints for useful data -->
@@ -797,6 +770,6 @@
       lower="-2.1"
       upper="2.1"
-      effort="0"
-      velocity="0" />
+      effort="8.85"
+      velocity="3.14" />
   </joint>
   <link name="Upper_Arm_2">
@@ -867,6 +840,6 @@
       lower="-0.1"
       upper="3.45"
-      effort="0"
-      velocity="0" />
+      effort="8.85"
+      velocity="3.14" />
   </joint>
   <link name="Lower_Arm_2">
@@ -928,5 +901,5 @@
     <child link="Lower_Arm_2" />
     <axis xyz="1 0 0" />
-    <limit lower="-0.2" upper="3.14159" effort="0" velocity="0" />
+    <limit lower="-0.2" upper="3.14159" effort="8.85" velocity="3.14" />
   </joint>
   <link name="Wrist_Pitch_Roll_2">
@@ -988,6 +961,6 @@
       lower="-1.8"
       upper="1.8"
-      effort="0"
-      velocity="0" />
+      effort="8.85"
+      velocity="3.14" />
   </joint>
   <link name="Fixed_Jaw_2">
@@ -1026,20 +999,11 @@
       </material>
     </visual>
-    <collision>
-      <origin
-        xyz="0 0 0"
-        rpy="0 0 0" />
-      <geometry>
-        <mesh
-          filename="package://xlerobot_gazebo/meshes/Fixed_Jaw_part1.ply" />
-      </geometry>
-    </collision>
-    <collision>
-      <origin
-        xyz="0 0 0"
-        rpy="0 0 0" />
-      <geometry>
-        <mesh
-          filename="package://xlerobot_gazebo/meshes/Fixed_Jaw_part2.ply" />
+    <!-- Simplified collision keeps the gripper movable in Gazebo. -->
+    <collision>
+      <origin
+        xyz="0.008 -0.044 0"
+        rpy="0 0 0" />
+      <geometry>
+        <box size="0.026 0.088 0.028" />
       </geometry>
     </collision>
@@ -1050,5 +1014,5 @@
     <child link="Fixed_Jaw_2" />
     <axis xyz="0 -1 0" />
-    <limit lower="-3.14159" upper="3.14159" effort="0" velocity="0" />
+    <limit lower="-3.14159" upper="3.14159" effort="8.85" velocity="3.14" />
   </joint>
   <link name="Moving_Jaw_2">
@@ -1077,27 +1041,8 @@
     <collision>
       <origin
-        xyz="0 0 0"
-        rpy="0 0 0" />
-      <geometry>
-        <mesh
-          filename="package://xlerobot_gazebo/meshes/Moving_Jaw_part1.ply" />
-      </geometry>
-    </collision>
-    <collision>
-      <origin
-        xyz="0 0 0"
-        rpy="0 0 0" />
-      <geometry>
-        <mesh
-          filename="package://xlerobot_gazebo/meshes/Moving_Jaw_part2.ply" />
-      </geometry>
-    </collision>
-    <collision>
-      <origin
-        xyz="0 0 0"
-        rpy="0 0 0" />
-      <geometry>
-        <mesh
-          filename="package://xlerobot_gazebo/meshes/Moving_Jaw_part3.ply" />
+        xyz="-0.003 -0.048 0"
+        rpy="0 0 0" />
+      <geometry>
+        <box size="0.018 0.072 0.02" />
       </geometry>
     </collision>
@@ -1108,5 +1053,6 @@
     <child link="Moving_Jaw_2" />
     <axis xyz="0 0 1" />
-    <limit lower="0" upper="1.7" effort="0" velocity="0" />
+    <dynamics damping="0.2" friction="0.0" />
+    <limit lower="-3.14159" upper="3.14159" effort="8.85" velocity="3.14" />
   </joint>
   <!-- fake joints for useful data -->
