Commit message: feat: Replace OmniWheelDriveController with custom kinematics
The ros2 omni_wheel_drive_controller didn't work correctly with
our 0°/120°/240° wheel layout. Replaced with:

- ForwardCommandController for direct wheel velocity control
- omni_twist_to_wheels.py: body twist → wheel velocities with
  rate limiting and envelope enforcement (inverse kinematics)
- omni_wheel_odometry.py: wheel joint states → odometry + TF
  (forward kinematics)

Also switched wheel collision from cylinder to sphere — the
standard Gazebo omni-wheel approach. Isotropic friction lets the
velocity controller drive correct wheel speeds while the body
slides freely in any direction.

Co-Authored-By: Claude Opus 4.6 (1M context) <noreply@anthropic.com>

File: src/xlerobot_gazebo/urdf/xlerobot.urdf.xacro (robot description, xacro)
@@ -132,7 +132,6 @@
       </visual>
       <collision>
-        <origin xyz="0 0 0" rpy="1.57079632679 0 0"/>
         <geometry>
-          <cylinder radius="${omni_wheel_radius}" length="${omni_wheel_width}"/>
+          <sphere radius="${omni_wheel_radius}"/>
         </geometry>
       </collision>
@@ -145,9 +144,10 @@
       <dynamics damping="0.05" friction="0.0"/>
     </joint>
-    <!-- Omni-wheel friction: near-zero along axle (roller slide), high perpendicular (drive). -->
+    <!-- Sphere collision with uniform friction simulates omni-wheel rollers:
+         the velocity controller drives the correct wheel speeds while the
+         isotropic contact allows the body to slide in any direction. -->
     <gazebo reference="wheel_${index}_link">
-      <mu1>0.001</mu1>
-      <mu2>1.5</mu2>
-      <fdir1>0 1 0</fdir1>
+      <mu1>1.0</mu1>
+      <mu2>1.0</mu2>
     </gazebo>
   </xacro:macro>

Commit message: fix: Fix omni wheel friction, body alignment, and teleop controls
- Fix omni wheel friction model: correct fdir1 direction for collision
  frame, reduce roller friction (mu1=0.001), increase lateral slip
  compliance (1.0) for proper omni-directional sliding
- Fix raskog body visual: correct swapped X/Y offset and 90° yaw
  misrotation so cart aligns with arms and wheels
- Fix forward direction: set wheel_offset=π so IK forward matches
  robot's visual front (arms/camera face -X)
- Improve keyboard teleop: unified speed parameter for all axes,
  independent per-axis keys for combined motion (W+A = diagonal),
  swap Q/E signs to match visual rotation, increase command timeout
  to 0.5s to prevent interruption during key hold
- Consolidate omni IK into base_twist_utils shared functions
- Add duplicate sim detection to launch scripts
- Add omni kinematics unit tests

Co-Authored-By: Claude Opus 4.6 (1M context) <noreply@anthropic.com>

File: src/xlerobot_gazebo/urdf/xlerobot.urdf.xacro (robot description, xacro)
@@ -4,4 +4,9 @@
   <xacro:property name="omni_wheel_radius" value="0.0508"/>
   <xacro:property name="omni_wheel_width" value="0.028"/>
+  <xacro:property name="omni_mu_free" value="0.001"/>
+  <xacro:property name="omni_mu_drive" value="1.5"/>
+  <xacro:property name="omni_slip_free" value="1.0"/>
+  <xacro:property name="omni_slip_drive" value="0.005"/>
+  <xacro:property name="omni_wheel_normal_force" value="260.0"/>
   <material name="white">
     <color rgba="0.3 0.3 0.3 1" />
@@ -65,5 +70,5 @@
     <visual name="raskog">
       <origin
-        xyz="-0.01668 0.502 0.895"
+        xyz="-0.01498 0.50143 0.895"
         rpy="1.5708 0 0" />
       <geometry>
@@ -75,5 +80,5 @@
     <visual name="raskogwheel1">
       <origin
-        xyz="-0.01668 0.502 0.895"
+        xyz="-0.01498 0.50143 0.895"
         rpy="1.5708 0 0" />
       <geometry>
@@ -85,5 +90,5 @@
     <visual name="raskogwheel2">
       <origin
-        xyz="-0.01668 0.502 0.895"
+        xyz="-0.01498 0.50143 0.895"
         rpy="1.5708 0 0" />
       <geometry>
@@ -132,6 +137,7 @@
       </visual>
       <collision>
+        <origin xyz="0 0 0" rpy="1.57079632679 0 0"/>
         <geometry>
-          <sphere radius="${omni_wheel_radius}"/>
+          <cylinder radius="${omni_wheel_radius}" length="${omni_wheel_width}"/>
         </geometry>
       </collision>
@@ -144,10 +150,13 @@
       <dynamics damping="0.05" friction="0.0"/>
     </joint>
-    <!-- Sphere collision with uniform friction simulates omni-wheel rollers:
-         the velocity controller drives the correct wheel speeds while the
-         isotropic contact allows the body to slide in any direction. -->
+    <!-- Omni-wheel friction: low along roller-slide direction, high in drive direction.
+         fdir1 is in the collision frame. The collision cylinder is rotated 90° around X
+         (rpy="π/2 0 0"), so collision Z = link Y (the axle / roller-slide direction).
+         mu1 (along fdir1) is near-zero for free roller sliding.
+         mu2 (perpendicular) is high for drive grip. -->
     <gazebo reference="wheel_${index}_link">
-      <mu1>1.0</mu1>
-      <mu2>1.0</mu2>
+      <mu1>${omni_mu_free}</mu1>
+      <mu2>${omni_mu_drive}</mu2>
+      <fdir1>0 0 1</fdir1>
     </gazebo>
   </xacro:macro>
@@ -1375,4 +1384,24 @@
       <parameters>$(arg controllers_file)</parameters>
     </plugin>
+    <plugin filename="gz-sim-wheel-slip-system" name="gz::sim::systems::WheelSlip">
+      <wheel link_name="wheel_0_link">
+        <slip_compliance_lateral>${omni_slip_free}</slip_compliance_lateral>
+        <slip_compliance_longitudinal>${omni_slip_drive}</slip_compliance_longitudinal>
+        <wheel_normal_force>${omni_wheel_normal_force}</wheel_normal_force>
+        <wheel_radius>${omni_wheel_radius}</wheel_radius>
+      </wheel>
+      <wheel link_name="wheel_1_link">
+        <slip_compliance_lateral>${omni_slip_free}</slip_compliance_lateral>
+        <slip_compliance_longitudinal>${omni_slip_drive}</slip_compliance_longitudinal>
+        <wheel_normal_force>${omni_wheel_normal_force}</wheel_normal_force>
+        <wheel_radius>${omni_wheel_radius}</wheel_radius>
+      </wheel>
+      <wheel link_name="wheel_2_link">
+        <slip_compliance_lateral>${omni_slip_free}</slip_compliance_lateral>
+        <slip_compliance_longitudinal>${omni_slip_drive}</slip_compliance_longitudinal>
+        <wheel_normal_force>${omni_wheel_normal_force}</wheel_normal_force>
+        <wheel_radius>${omni_wheel_radius}</wheel_radius>
+      </wheel>
+    </plugin>
   </gazebo>
 </robot>
